File: Fichier_PCB/PCM1804/PCM1804.kicad_sch (KiCad schematic)
At the start: 14 parts

Commit message: kicad pour pcm1804 version 1 fini
Parts:
- removed C? (x4): 10uF, symbol Device:C_Polarized
- removed C? (x2): 0.1uF, symbol Device:C_Polarized
- removed C? (x4): 0.1uF, symbol Device:C
- removed IC?: PCM1804, DB_R-PDSO-G28, symbol PCM1804:PCM1804
- removed R? (x2): 10k, symbol Device:R
- removed RN?: R_Pack10K, symbol Device:R_Pack07
- added C? (x4): 10uF, symbol Device:C_Polarized
- added C? (x4): 0.1uF, symbol Device:C
- added C? (x2): 0.1uF, symbol Device:C_Polarized
- added IC?: PCM1804, DB_R-PDSO-G28, symbol PCM1804:PCM1804
- added R? (x2): 10k, symbol Device:R
- added RN?: R_Pack10K, symbol Device:R_Pack07
Connections:
- net 3V3: now also C?.1, C?.1, IC?.14 (VDD), RN?.11 (R4.2), RN?.12 (R3.2), RN?.14 (R1.2), RN?.8 (R7.2)
- net 5V: now also C?.1, C?.1, IC?.22 (VCC)
- net BCK: now also IC?.16 (BCK/DSDL)
- net DATA: now also IC?.15 (DATA/DSDR)
- net GND: now also C?.1, C?.1, C?.2, C?.2, C?.2, C?.2, C?.2, C?.2, C?.2, C?.2, IC?.13 (DGND), IC?.2 (AGNDL), IC?.23 (AGND), IC?.27 (AGNDR), R?.2, R?.2, RN?.10 (R5.2), RN?.13 (R2.2), RN?.9 (R6.2)
- net LRCK: now also IC?.17 (LRCK/DSDBCK)
- net RST: now also IC?.19 (~{RST})
- net SCKL: now also IC?.18 (SCKI)
- net VCOM: now also C?.1, IC?.3 (VCOML)
- net VIN+: now also IC?.4 (VINL+)
- net VIN-: now also IC?.5 (VINL-)
- new net: C?.1, C?.2, IC?.28 (VREFR)
- new net: IC?.12 (BYPAS), RN?.1 (R1.1)
- new net: IC?.11 (OSR2), RN?.2 (R2.1)
- new net: IC?.10 (OSR1), RN?.3 (R3.1)
- new net: IC?.9 (OSR0), RN?.4 (R4.1)
- new net: IC?.8 (S/~{M}), RN?.5 (R5.1)
- new net: IC?.7 (FMT1), RN?.6 (R6.1)
- new net: IC?.6 (FMT0), RN?.7 (R7.1)
- new net: C?.1, C?.2, IC?.1 (VREFL)
- new net: IC?.24 (VINR-), R?.1
- new net: C?.1, IC?.26 (VCOMR)
- new net: IC?.25 (VINR+), R?.1
