File: Fichier_PCB/Ecout-Terre_PCB_V1/Ecout-Terre_PCB_V1.kicad_pcb (KiCad board)
At the start: 4 copper layers, 92 x 86 mm, 111 parts, among them J1 USB_C_Receptacle_USB2.0, J10 Micro_SD_Card, J11 Test_10V, J12 Conn_test_ampli, J13 Conn_GPS, J14 AudioJack_Mono, J2 Pile, J4 Test_5V, J5 Conn_Alim, J6 Test_3V3, J7 Conn_ESP, J8 Conn_ESP, J9 Sortie_alim, Q1 CSD16327Q3, U1 TS3480CX33RFG, U2 MC33269, U3 LM3478, U4 PCM1804, U5 TL072, U6 LM386, U7 74LVT04, Y1 7V-22.5792MAHV-T

Commit message: Envoie de code et correction PCB
Routing:
- net GND: track 1052.8 -> 1056.0 mm
Changed lines of the file:
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@@
   (segment (start 165.9 134.225) (end 146.235733 114.560733) (width 0.33) (layer "In1.Cu") (net 2))
   (segment (start 167.817744 75.467744) (end 165.25 72.9) (width 0.33) (layer "In1.Cu") (net 2))
+  (segment (start 142.342744 114.560733) (end 140.107011 112.325) (width 0.33) (layer "In1.Cu") (net 2))
   (segment (start 132.298731 125.475) (end 133.184511 124.58922) (width 0.33) (layer "In1.Cu") (net 2))
   (segment (start 165.9 134.225) (end 169.032255 131.092745) (width 0.33) (layer "In1.Cu") (net 2))
@@
   (segment (start 110.825 106.922421) (end 120.119877 97.627544) (width 0.33) (layer "In1.Cu") (net 2))
   (segment (start 120.119877 97.627544) (end 121.047349 97.627544) (width 0.33) (layer "In1.Cu") (net 2))
-  (segment (start 140.107011 112.325) (end 139.525 112.325) (width 0.33) (layer "In1.Cu") (net 2))
   (segment (start 122.625 117.175) (end 122.625 115.25) (width 0.33) (layer "In1.Cu") (net 2))
   (segment (start 128.545 70.5) (end 130.79142 68.25358) (width 0.33) (layer "In1.Cu") (net 2))
@@
   (segment (start 166.575 98.033477) (end 167.817744 96.790733) (width 0.33) (layer "In1.Cu") (net 2))
   (segment (start 123.285 134.435) (end 124.835 134.435) (width 0.33) (layer "In1.Cu") (net 2))
+  (segment (start 140.107011 112.325) (end 139.525 112.325) (width 0.33) (layer "In1.Cu") (net 2))
   (segment (start 114.325 125.475) (end 132.298731 125.475) (width 0.33) (layer "In1.Cu") (net 2))
   (segment (start 172.98952 71.25452) (end 173.7 71.965) (width 0.33) (layer "In1.Cu") (net 2))
