File: Fichier_PCB/Ecout-Terre_PCB_V2/9V_alim.kicad_sch (KiCad schematic)
At the start: 28 parts, among them J1 USB_C_Receptacle_USB2.0, J11 Test_10V, J2 Pile, J4 Test_5V, J6 Test_3V3, J9 Sortie_alim, Q1 CSD16327Q3, U1 TS3480CX33RFG, U2 MC33269, U3 LM3478

Commit message: Trace pcb
Parts:
- C8: footprint Capacitor_SMD:C_0805_2012Metric_Pad1.18x1.45mm_HandSolder -> Capacitor_SMD:C_0504_1310Metric_Pad0.83x1.28mm_HandSolder
Changed lines of the file:
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@@
       (effects (font (size 1.27 1.27)) (justify left))
     )
-    (property "Footprint" "Capacitor_SMD:C_0805_2012Metric_Pad1.18x1.45mm_HandSolder" (id 2) (at 122.8852 87.63 0)
+    (property "Footprint" "Capacitor_SMD:C_0504_1310Metric_Pad0.83x1.28mm_HandSolder" (id 2) (at 122.8852 87.63 0)
       (effects (font (size 1.27 1.27)) hide)
     )
